File: Jetson-AI-Cam-CopperPilot.kicad_pcb (KiCad board)
At the start: 8 copper layers, 78 x 55 mm, 326 parts, among them IC1 NCP380LSNAJAAT1G, IC11 SN74LV1T125DBVR, IC12 74HC00_TSSOP, IC13 SN74LVC1G126_SC-70, IC15 TPS7A0518P_SOT23-5, IC17 AT24CS01_SOT23, IC18 TPD8S009DSMR, IC2 TPD8S009DSMR, IC3 NCP380LSNAJAAT1G, IC4 TPS7A0518P_SOT23-5, IC5 FT232R_QFN, IC6 PCA9517ADP, IC7 HD3SS3220RNH, J1 HDMI-Micro-D_Molex_467561001, J10 Conn_FFC_Molex_5051101097, J11 USB-C_WE_632723300011, J12 Molex_PicoBlade_1x4_0533980471, J13 JST_SH_1x4_SM04B-SRSS-TB-LF-SN, J14 JST_SH_1x4_SM04B-SRSS-TB-LF-SN, J15 Bus_DDR4_SODIMM_CUSTOM_Jetson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, J2 DisplayPort-Mini_TE_2129320-3, J4 Conn_01x02, J5 USB-Micro-B_Molex_473460001, J9 USB-Micro-B_Molex_473460001, M2 Jetson-Nano, T1 BSS138PW, T2 BSS138PW, T3 BSS138PW, T4 BSS138PW, T5 BSS138PW, T6 BSS138PW, T7 BSS138PW, T8 BSS138PW, T9 BSS138PW, U1 LM3671MF-3.3_SOT, U10 TPS7A0528PDBVR, U11 TPS7A0512PDBVR, U2 LM62440-Q1, U3 SN74LXC1T45DBVR, U4 PCA9547_VQFN, U6 SIC477ED-T1-GE3, U7 MAX3051EKA, U8 74LVC1G07_SOT-753

Commit message: pcb: route Milestone 27 - /Supply/5V_SS microvia breakout to In5 (34 -> 33 unconnected)
Routing:
- net /Supply/5V_SS: track 0.00 -> 4.21 mm, vias 0 -> 2
Changed lines of the file:
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@@
+	)
+	(segment
+		(start 100.15 85.923)
+		(end 100.15 86.6)
+		(width 0.15)
+		(layer "B.Cu")
+		(net "/Supply/5V_SS")
+	)
+	(segment
+		(start 100.15 86.6)
+		(end 103.634 87.2)
+		(width 0.15)
+		(layer "In5.Cu")
+		(net "/Supply/5V_SS")
+	)
+	(via micro
+		(at 103.634 87.2)
+		(size 0.25)
+		(drill 0.1)
+		(layers "In5.Cu" "B.Cu")
+		(net "/Supply/5V_SS")
+	)
+	(via micro
+		(at 100.15 86.6)
+		(size 0.25)
+		(drill 0.1)
+		(layers "In5.Cu" "B.Cu")
+		(net "/Supply/5V_SS")
 	)
 	(segment
