File: display.kicad_sch (KiCad schematic)
At the start: 65 parts, among them IC11 SN74LV1T125DBVR, IC18 TPD8S009DSMR, IC2 TPD8S009DSMR, IC6 PCA9517ADP, J1 HDMI-Micro-D_Molex_467561001, J15 Bus_DDR4_SODIMM_CUSTOM_Jetson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, J2 DisplayPort-Mini_TE_2129320-3, T1 BSS138PW

Commit message: fix(sch): resolve all PWR_FLAG, label, and differential-corridor collisions on Display sheet (Page 5)
Remove duplicate TMDS_HPD label on J15E, relocate colliding PWR_FLAG symbols on J1/J2/IC2/top-left and hide flag text, move C73-C80/R1-R10/C39-C45/R98-R99 properties out of differential wire corridors, clean up R31/R32/T1, and delete stray off-sheet artifacts.

Co-Authored-By: CopperPilot <noreply@copperpilot.ai>
Other:
- note removed: "Text"
