File: supply.kicad_sch (KiCad schematic)
At the start: 0 parts

Commit message: feat: refactor schematics - remove Ethernet and M.2 NVMe, compact power entry J4, and integrate CAM_L and CAM_R stereo camera sensors
Parts:
- added C16, C18, C60: C_2u2_0402, jetson-footprints:C_0402_1005Metric, symbol jetson-symbols:C_2u2_0402
- added C17, C19, C21, C22: C_10u_1206_50V, jetson-footprints:C_1206_3216Metric, symbol jetson-symbols:C_10u_1206_50V
- added C20, C59, C64: C_47u_0805, jetson-footprints:C_0805_2012Metric, symbol jetson-symbols:C_47u_0805
- added C23, C55, C63, C81: C_10u_0603, jetson-footprints:C_0603_1608Metric, symbol jetson-symbols:C_10u_0603
- added C24: C_6p_0402, jetson-footprints:C_0402_1005Metric, symbol jetson-symbols:C_6p_0402
- added C25: C_10u_0805, jetson-footprints:C_0805_2012Metric, symbol jetson-symbols:C_10u_0805
- added C28: C_270p_25V_0402, jetson-footprints:C_0402_1005Metric, symbol jetson-symbols:C_270p_25V_0402
- added C41: C_47n_0402, jetson-footprints:C_0402_1005Metric, symbol jetson-symbols:C_47n_0402
- added C56: C_100n_50V_0402, jetson-footprints:C_0402_1005Metric, symbol jetson-symbols:C_100n_50V_0402
- added C57, C71, C83, C86, C88, C89: C_100n_0402, jetson-footprints:C_0402_1005Metric, symbol jetson-symbols:C_100n_0402
- added C58: C_33n_0402, jetson-footprints:C_0402_1005Metric, symbol jetson-symbols:C_33n_0402
- added C61, C82: C_1n2_50V_0402, jetson-footprints:C_0402_1005Metric, symbol jetson-symbols:C_1n2_50V_0402
- added C65, C84, C87: C_1u_0402, jetson-footprints:C_0402_1005Metric, symbol jetson-symbols:C_1u_0402
- added C85: C_4u7_0603, jetson-footprints:C_0603_1608Metric, symbol jetson-symbols:C_4u7_0603
- added D1, D9: ESD5B5_0ST1G, jetson-footprints:SOD-523_NP, symbol jetson-symbols:ESD5B5_0ST1G
- added D13: 1N4148WS, jetson-footprints:D_SOD-323F, symbol jetson-symbols:1N4148WS
- added D14: SMBJ33A, jetson-footprints:D_SMB, symbol jetson-symbols:SMBJ33A
- added F1, F2: F_1.25A_0603, jetson-footprints:F_0603_1608Metric, symbol jetson-symbols:F_1.25A_0603
- added F3: F_12A_1206, jetson-footprints:F_1206_3216Metric, symbol jetson-symbols:F_12A_1206
- added FB1: FB_10Z_10A_WE-MPSB_1206, jetson-footprints:FB_1206_3216Metric, symbol jetson-symbols:FB_10Z_10A_WE-MPSB_1206
- added FB3: FB_180Z_3.1A_WE-MPSB_0805, jetson-footprints:FB_0805_2012Metric, symbol jetson-symbols:FB_180Z_3.1A_WE-MPSB_0805
- added IC12: 74HC00_TSSOP, jetson-footprints:TSSOP-14_4.4x5mm_P0.65mm, symbol jetson-symbols:74HC00_TSSOP
- added IC13: SN74LVC1G126_SC-70, jetson-footprints:SC-70-5, symbol jetson-symbols:SN74LVC1G126_SC-70
- added IC4: TPS7A0518P_SOT23-5, jetson-footprints:SOT-23-5, symbol jetson-symbols:TPS7A0518P_SOT23-5
- added J12: Molex_PicoBlade_1x4_0533980471, jetson-footprints:Conn_Molex_PicoBlade_1x4_0533980471, symbol jetson-symbols:Molex_PicoBlade_1x4_0533980471
- added J4: Conn_01x02, jetson-footprints:PinHeader_1x02_P2.54mm_Vertical, symbol jetson-symbols:Conn_01x02
- added L1: L_2u2_8A_Coilcraft-XFL4020, jetson-footprints:L_Coilcraft-XFL4020, symbol jetson-symbols:L_2u2_8A_Coilcraft-XFL4020
- added L4: L_3u3_9.2A_Vishay-IHLP-3232DZ-01, jetson-footprints:L_Vishay-IHLP3232DZ, symbol jetson-symbols:L_3u3_9.2A_Vishay-IHLP-3232DZ-01
- added L5, L6: L_2u2_1.6A_1210, jetson-footprints:L_1210_3225Metric, symbol jetson-symbols:L_2u2_1.6A_1210
- added R117: R_52k3_0402, jetson-footprints:R_0402_1005Metric, symbol jetson-symbols:R_52k3_0402
- added R118, R91, R96: R_100k_0402, jetson-footprints:R_0402_1005Metric, symbol jetson-symbols:R_100k_0402
- added R119: R_44k2_0402, jetson-footprints:R_0402_1005Metric, symbol jetson-symbols:R_44k2_0402
- added R120, R39, R44, R46, R52, R95: R_10k_0402, jetson-footprints:R_0402_1005Metric, symbol jetson-symbols:R_10k_0402
- added R130, R48, R76, R92, R93: R_0R_0402, jetson-footprints:R_0402_1005Metric, symbol jetson-symbols:R_0R_0402
- added R16, R36, R45, R87: R_1k_0402, jetson-footprints:R_0402_1005Metric, symbol jetson-symbols:R_1k_0402
- added R70: R_100R_0402, jetson-footprints:R_0402_1005Metric, symbol jetson-symbols:R_100R_0402
- added R74: R_2k_0402, jetson-footprints:R_0402_1005Metric, symbol jetson-symbols:R_2k_0402
- added R75: R_316k_0402, jetson-footprints:R_0402_1005Metric, symbol jetson-symbols:R_316k_0402
- added R77: R_60k4_0402, jetson-footprints:R_0402_1005Metric, symbol jetson-symbols:R_60k4_0402
- added R84, R86: R_200k_0402, jetson-footprints:R_0402_1005Metric, symbol jetson-symbols:R_200k_0402
- added R85: R_470k_0402, jetson-footprints:R_0402_1005Metric, symbol jetson-symbols:R_470k_0402
- added R89: R_3R3_0402, jetson-footprints:R_0402_1005Metric, symbol jetson-symbols:R_3R3_0402
- added R90: R_26k7_0402, jetson-footprints:R_0402_1005Metric, symbol jetson-symbols:R_26k7_0402
- added R94: R_8k66_0402, jetson-footprints:R_0402_1005Metric, symbol jetson-symbols:R_8k66_0402
- added T3: BSS138PW, jetson-footprints:SC70-3, symbol jetson-symbols:BSS138PW
- added TP11, TP12, TP15, TP16, TP40, TP41, TP42, TP44, TP47, TP5, TP8: TP_1.5mm_SMD, jetson-footprints:TP_SMD_1.5mm, symbol jetson-symbols:TP_1.5mm_SMD
- added U1, U5: LM3671MF-3.3_SOT, jetson-footprints:SOT-23-5, symbol jetson-symbols:LM3671MF-3.3_SOT
- added U2: LM62440-Q1, jetson-footprints:VQFN-HR-14_3.5x4mm, symbol jetson-symbols:LM62440-Q1
- added U3: SN74LXC1T45DBVR, jetson-footprints:SOT-23-6, symbol jetson-symbols:SN74LXC1T45DBVR
- added U6: SIC477ED-T1-GE3, jetson-footprints:SIC47XED-T1-GE3, symbol jetson-symbols:SIC477ED-T1-GE3
Connections:
- new net: IC12.10 (3B), IC12.11 (~{4Y}), IC12.9 (3A)
- new net: IC12.2 (1B), IC12.6 (~{2Y}), R16.2
- new net: IC12.8 (~{3Y}), R130.2
- new net: F3.1, J4.1 (Pin_1)
- new net: IC4.3 (EN), R92.2
- new net: C23.1, F1.1, L5.2, TP5.1, U1.4 (FB)
- new net: C55.1, F2.1, L6.2, TP8.1, U5.4 (FB)
- new net: C57.1, R89.1
- new net: R39.2, U1.3 (EN)
- new net: L5.1, U1.5 (SW)
- new net: R52.2, U5.3 (EN)
- new net: L6.1, U5.5 (SW)
- new net: C61.1, R93.1, U6.20 (V_{SNS})
- new net: R70.1, U2.13 (RBOOT)
- new net: C24.2, R45.1
- new net: C28.1, R75.2
- new net #RESET: R39.1, R44.1, R52.1, R92.1
- new net #SHUTDOWN_REQ: IC12.4 (2A), R86.2
- new net 1V8_SYS: C65.1, C86.1, IC4.5 (VOUT), R95.1, T3.1 (G), TP47.1, U3.1 (VCCA), U3.5 (DIR)
- new net 3V3_EN: R44.2, U2.7 (EN)
- new net 3V3_FB: R118.2, R119.1, R45.2, R48.2, U2.4 (FB)
- new net 3V3_FFC1: F1.2
- new net 3V3_FFC2: F2.2
- new net 3V3_R_C_BOOT: C89.2, R70.2, U2.14 (CBOOT)
- new net 3V3_SW: C89.1, L1.1, U2.10 (SW)
- new net 3V3_SYS: C20.1, C24.1, C25.1, D1.2 (A), L1.2, R118.1, R48.1, U2.1 (BIAS)
- new net 3V3_VCC: C87.1, U2.2 (VCC)
- new net 3V3_VIN: C19.1, C21.1, FB3.2, U2.12 (VIN), U2.8 (VIN)
- new net 5V0_SYS: C16.1, C18.1, C59.1, C60.1, C64.1, C71.1, C81.1, C82.2, C83.1, C88.1, D9.2 (A), IC12.14 (VCC), IC13.1 (OE), IC13.5 (VCC), IC4.1 (VIN), J12.2, L4.2, R117.1, R16.1, R36.1, R46.1, R84.1, R86.1, R93.2, TP41.1, TP42.1, U1.1 (V_{IN}), U3.6 (VCCB), U5.1 (V_{IN})
- new net 5V_BOOT: C57.2, U6.4 (BOOT)
- new net 5V_COMP: R75.1, U6.21 (NC)
- new net 5V_EN: R91.1, TP15.1, U6.3 (EN)
- new net 5V_FB: R117.2, R120.1, U6.22 (V_{FB})
- new net 5V_FSW: R90.1, U6.24 (f_{SW})
- new net 5V_ILIM: R76.2, R77.1, U6.25 (I_{LIMIT})
- new net 5V_MODE: R74.1, U6.27 (MODE)
- new net 5V_PHASE: R89.2, U6.5 (PHASE), U6.6 (PHASE)
- new net 5V_SNS: C61.2, C82.1, R94.2
- new net 5V_SS: C58.1, U6.19 (SS)
- new net 5V_SW: L4.1, R94.1, U6.12 (SW), U6.13 (SW), U6.14 (SW)
- new net 5V_VIN: C17.1, C22.1, C56.1, FB1.2, R91.2, TP11.1, U6.1 (V_{CIN}), U6.7 (V_{IN}), U6.8 (V_{IN})
- new net FAN_PMW_5V: J12.4, U3.4 (B)
- new net FAN_PWM: U3.3 (A)
- new net FAN_TACH: R95.2, T3.2 (S)
- new net FAN_TACH_5V: J12.3, R46.2, T3.3 (D)
- new net GND: C16.2, C17.2, C18.2, C19.2, C20.2, C21.2, C22.2, C23.2, C25.2, C28.2, C41.2, C55.2, C56.2, C58.2, C59.2, C60.2, C63.2, C64.2, C65.2, C71.2, C81.2, C83.2, C84.2, C85.2, C86.2, C87.2, C88.2, D1.1 (C), D14.2 (A), D9.1 (C), IC12.7 (GND), IC13.3 (GND), IC4.2 (GND), J12.1, J4.2 (Pin_2), R119.2, R120.2, R74.2, R77.2, R90.2, TP12.1, TP44.1, U1.2 (GND), U2.11 (PGND), U2.3 (AGND), U2.6 (MODE), U2.9 (PGND), U3.2 (GND), U5.2 (GND), U6.10 (PGND), U6.11 (PGND), U6.17 (PGND), U6.23 (AGND), U6.28 (AGND), U6.9 (PGND)
- new net PWR_EN: IC13.4 (Y), R130.1
- new net PWR_GOOD: R87.1, R96.1, TP40.1, U6.2 (P_{GOOD})
- new net Q: D13.1 (C), IC12.3 (~{1Y}), IC12.5 (2B), R36.2, R85.1
- new net QDEL: C63.1, D13.2 (A), IC12.12 (4A), IC12.13 (4B), IC13.2 (A), R85.2, R87.2
- new net VDD_5V_DCDC: C84.1, R76.1, R96.2, U6.26 (V_{DD})
- new net VDRV_5V_DCDC: C85.1, U6.16 (V_{DRV})
- new net VIN: D14.1 (C), F3.2, FB1.1, FB3.1, TP16.1
- new net \~{PWR_SET}: C41.1, IC12.1 (1A), R84.2
- no-connect marks 0 -> 5
Other:
- note added: "#PWR_RST"
- note added: "0.8V typ"
- note added: "12A"
- note added: "1MHz"
- note added: "3V3 DC/DC"
- note added: "3V3 FFC 1&2"
- note added: "3V3/3.5A"
- note added: "52k3 -> 4.98V"
- note added: "52k5 -> 5.0V"
- note added: "5V DC/DC"
- note added: "5V/8A"
- note added: "9...36 VDC"
- note added: "FAN 5V"
- note added: "Note: Place close to the feedback resistors"
- note added: "Note: SIC477 can be substituted with SIC472. If so: R75, R77, R94, C28, C61, C82 are populated, R76, R93 are DNP"
- note added: "Power Supply"
- note added: "Power input"
- note added: "Power save mode enabled, VDD, VDRVPre-reg on"
- note added: "Power sequencer"
- note added: "R_FB_H = R_FB_L * (V_OUT - V_FB) / V_FB 10k * (5 - 0.8) / 0.8 = 52K5"
- note added: "System 1V8"
- note added: "Text"

Commit message: refactor(pcb,sch): remove all 36 test points and prune associated stub tracks
Parts:
- removed TP11, TP12, TP15, TP16, TP40, TP41, TP42, TP44, TP47, TP5, TP8: TP_1.5mm_SMD, jetson-footprints:TP_SMD_1.5mm, symbol jetson-symbols:TP_1.5mm_SMD

Commit message: fix(schematic): remediate camera clocking, power sequencing, and ERC errors
- Connect Sony IMX219 master clocks (CAM0/1_MCLK) from SoM pins 116/122
- Connect independent PWDN hardware resets from SoM pins 114/120
- Isolate sensor I2C channels (CAM0/1_SCL/SDA) downstream of PCA9547
- Upgrade U11 digital core LDO to TLV75512PDBVR (500mA rating)
- Ground R132 to enable serial EEPROM write-protect
- Connect 3V3_SYS power rail to CAN transceiver U7 and fuse F5
- Eliminate dangling global labels across all sheets
- Configure 25 mil connection grid and achieve 0 ERC errors
Changed lines of the file:
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@@
-	(symbol
-		(lib_id "jetson-symbols:GND")
-		(at 121.285 85.09 0)
-		(unit 1)
-		(body_style 1)
-		(exclude_from_sim no)
-		(in_bom yes)
-		(on_board yes)
-		(in_pos_files yes)
-		(dnp no)
-		(fields_autoplaced yes)
-		(property "Reference" "#GND_0145"
-			(at 121.285 85.09 0)
-			(hide yes)
-			(show_name no)
-			(do_not_autoplace no)
-			(effects
-				(font
-					(size 1.27 1.27)
-				)
-				(justify left)
-			)
-		)
-		(property "Value" "GND"
-			(at 121.285 89.535 0)
-			(show_name no)
-			(do_not_autoplace no)
-			(effects
-				(font
-					(size 1.27 1.27)
-				)
-			)
-		)
-		(property "Footprint" ""
-			(at 121.285 85.09 0)
-			(hide yes)
-			(show_name no)
-			(do_not_autoplace no)
-			(effects
-				(font
-					(size 1.27 1.27)
-				)
-				(justify left)
-			)
-		)
-		(property "Datasheet" ""
-			(at 121.285 85.09 0)
-			(hide yes)
-			(show_name no)
-			(do_not_autoplace no)
-			(effects
-				(font
-					(size 1.27 1.27)
-				)
-				(justify left)
-			)
-		)
-		(property "Description" ""
-			(at 121.285 85.09 0)
-			(show_name no)
-			(do_not_autoplace no)
-			(effects
-				(font
-					(size 1.27 1.27)
-				)
-			)
-		)
-		(property "License" "Apache-2.0"
-			(at 130.175 95.25 0)
-			(hide yes)
-			(show_name no)
-			(do_not_autoplace no)
-			(effects
-				(font
-					(size 1.27 1.27)
-					(thickness 0.15)
-				)
-				(justify left bottom)
-			)
-		)
-		(pin "1"
-		)
-		(instances
-			(project "Jetson-AI-Cam-CopperPilot"
-				(path "/9df9f3e2-e127-4935-b743-4d95c8ce9b2e/00000000-0000-0000-0000-0000608dc6e9"
-					(reference "#GND_0145")
-					(unit 1)
-				)
-			)
-		)
-	)
 	(symbol
 		(lib_id "jetson-symbols:GND")

Commit message: fix(supply): ground J12 tabs, DNP U5 aux buck, add VIN/VSNS PWR_FLAG, and prune 10 wire stubs
Parts:
- C18, C55, F2, L6, R52, U5: now not fitted; now left out of the parts list
Connections:
- net GND: now also J12.MP1, J12.MP2
Changed lines of the file:
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@@
 		(body_style 1)
 		(exclude_from_sim no)
-		(in_bom yes)
-		(on_board yes)
+		(in_bom no)
+		(on_board no)
 		(in_pos_files yes)
-		(dnp no)
+		(dnp yes)
 		(fields_autoplaced yes)
 		(property "Reference" "U5"
@@
 		(body_style 1)
 		(exclude_from_sim no)
-		(in_bom yes)
-		(on_board yes)
+		(in_bom no)
+		(on_board no)
 		(in_pos_files yes)
-		(dnp no)
+		(dnp yes)
 		(fields_autoplaced yes)
 		(property "Reference" "F2"
@@
 		(body_style 1)
 		(exclude_from_sim no)
-		(in_bom yes)
-		(on_board yes)
+		(in_bom no)
+		(on_board no)
 		(in_pos_files yes)
-		(dnp no)
+		(dnp yes)
 		(fields_autoplaced yes)
 		(property "Reference" "L6"
@@
 		(body_style 1)
 		(exclude_from_sim no)
-		(in_bom yes)
-		(on_board yes)
+		(in_bom no)
+		(on_board no)
 		(in_pos_files yes)
-		(dnp no)
+		(dnp yes)
 		(fields_autoplaced yes)
 		(property "Reference" "C55"
@@
 		(body_style 1)
 		(exclude_from_sim no)
-		(in_bom yes)
-		(on_board yes)
+		(in_bom no)
+		(on_board no)
 		(in_pos_files yes)
-		(dnp no)
+		(dnp yes)
 		(property "Reference" "R52"
 			(at 53.34 218.44 0)
@@
 		(body_style 1)
 		(exclude_from_sim no)
-		(in_bom yes)
-		(on_board yes)
+		(in_bom no)
+		(on_board no)
 		(in_pos_files yes)
-		(dnp no)
+		(dnp yes)
 		(fields_autoplaced yes)
 		(property "Reference" "C18"
@@
 	)	(wire
 		(pts
-			(xy 102.235 214.63) (xy 102.235 216.535)
-		)
-		(stroke
-			(width 0)
-			(type default)
-		)
-	)	(wire
-		(pts
 			(xy 93.345 137.795) (xy 107.95 137.795)
 		)
@@
 	)	(wire
 		(pts
-			(xy 354.33 100.33) (xy 351.79 100.33)
-		)
-		(stroke
-			(width 0)
-			(type default)
-		)
-	)	(wire
-		(pts
 			(xy 40.64 85.725) (xy 40.64 86.995)
 		)
@@
 	)	(wire
 		(pts
-			(xy 102.235 188.595) (xy 102.235 190.5)
-		)
-		(stroke
-			(width 0)
-			(type default)
-		)
-	)	(wire
-		(pts
 			(xy 108.585 46.99) (xy 117.475 46.99)
 		)
@@
 	)	(wire
 		(pts
-			(xy 78.105 57.785) (xy 80.01 57.785)
-		)
-		(stroke
-			(width 0)
-			(type default)
-		)
-	)	(wire
-		(pts
 			(xy 267.97 46.99) (xy 267.97 52.07)
 		)
@@
 	)	(wire
 		(pts
-			(xy 252.73 250.19) (xy 255.905 250.19)
-		)
-		(stroke
-			(width 0)
-			(type default)
-		)
-	)	(wire
-		(pts
 			(xy 110.49 216.535) (xy 102.235 216.535)
 		)
@@
 	)	(wire
 		(pts
-			(xy 212.725 192.405) (xy 212.725 194.31)
-		)
-		(stroke
-			(width 0)
-			(type default)
-		)
-	)	(wire
-		(pts
 			(xy 93.345 142.875) (xy 95.25 142.875)
 		)
@@
 	)	(wire
 		(pts
-			(xy 214.63 45.72) (xy 214.63 46.99)
-		)
-		(stroke
-			(width 0)
-			(type default)
-		)
-	)	(wire
-		(pts
 			(xy 279.4 83.82) (xy 269.24 83.82)
 		)
@@
 	)	(wire
 		(pts
-			(xy 377.19 59.69) (xy 379.73 59.69)
-		)
-		(stroke
-			(width 0)
-			(type default)
-		)
-	)	(wire
-		(pts
 			(xy 130.175 149.225) (xy 139.7 149.225)
 		)
@@
 	)	(wire
 		(pts
-			(xy 121.285 73.025) (xy 121.285 74.295)
-		)
-		(stroke
-			(width 0)
-			(type default)
-		)
-	)	(wire
-		(pts
 			(xy 119.38 60.325) (xy 118.11 60.325)
 		)
@@
 	)	(wire
 		(pts
-			(xy 80.01 45.72) (xy 80.01 46.99)
-		)
-		(stroke
-			(width 0)
-			(type default)
-		)
-	)	(wire
-		(pts
 			(xy 293.37 71.12) (xy 275.59 71.12)
 		)
@@
 					(unit 1)
 				)
+			)
+		)
+	)
+	(symbol
+		(lib_id "jetson-symbols:GND")
+		(at 346.075 129.54 0)
+		(unit 1)
+		(body_style 1)
+		(exclude_from_sim no)
+		(in_bom yes)
+		(on_board yes)
+		(in_pos_files yes)
+		(dnp no)
+		(property "Reference" "#PWR_J12_MP1"
+			(at 346.075 127.0 0)
+			(hide yes)
+			(effects (font (size 1.27 1.27)))
+		)
+		(property "Value" "GND"
+			(at 346.075 127.0 0)
+			(hide yes)
+			(effects (font (size 1.27 1.27)))
+		)
+		(pin "1")
+		(instances
+			(project "Jetson-AI-Cam-CopperPilot"
+				(path "/9df9f3e2-e127-4935-b743-4d95c8ce9b2e/00000000-0000-0000-0000-0000608dc6e9"
+					(reference "#PWR_J12_MP1")
+					(unit 1)
+				)
+			)
+		)
+	)
+	(symbol
+		(lib_id "jetson-symbols:GND")
+		(at 346.075 127.0 0)
+		(unit 1)
+		(body_style 1)
+		(exclude_from_sim no)
+		(in_bom yes)
+		(on_board yes)
+		(in_pos_files yes)
+		(dnp no)
+		(property "Reference" "#PWR_J12_MP2"
+			(at 346.075 154.94 0)
+			(hide yes)
+			(effects (font (size 1.27 1.27)))
+		)
+		(property "Value" "GND"
+			(at 346.075 154.94 0)
+			(hide yes)
+			(effects (font (size 1.27 1.27)))
+		)
+		(pin "1")
+		(instances
+			(project "Jetson-AI-Cam-CopperPilot"
+				(path "/9df9f3e2-e127-4935-b743-4d95c8ce9b2e/00000000-0000-0000-0000-0000608dc6e9"
+					(reference "#PWR_J12_MP2")
+					(unit 1)
+				)
+			)
+		)
+	)
+	(symbol
+		(lib_id "jetson-symbols:PWR_FLAG")
+		(at 73.025 132.715 0)
+		(unit 1)
+		(body_style 1)
+		(exclude_from_sim no)
+		(in_bom yes)
+		(on_board yes)
+		(in_pos_files yes)
+		(dnp no)
+		(property "Reference" "#FLG_U2_VIN"
+			(at 73.025 130.175 0)
+			(effects (font (size 1.27 1.27)))
+		)
+		(property "Value" "PWR_FLAG"
+			(at 73.025 135.255 0)
+			(effects (font (size 1.27 1.27)))
+		)
+		(pin "1")
+		(instances
+			(project "Jetson-AI-Cam-CopperPilot"
+				(path "/9df9f3e2-e127-4935-b743-4d95c8ce9b2e/00000000-0000-0000-0000-0000608dc6e9"
+					(reference "#FLG_U2_VIN")
+					(unit 1)
+				)
+			)
+		)
+	)
+	(symbol
+		(lib_id "jetson-symbols:PWR_FLAG")
+		(at 116.205 62.865 0)
+		(unit 1)
+		(body_style 1)
+		(exclude_from_sim no)
+		(in_bom yes)
+		(on_board yes)
+		(in_pos_files yes)
+		(dnp no)
+		(property "Reference" "#FLG_U6_VSNS"
+			(at 116.205 60.325 0)
+			(effects (font (size 1.27 1.27)))
+		)
+		(property "Value" "PWR_FLAG"
+			(at 116.205 65.405 0)
+			(effects (font (size 1.27 1.27)))
+		)
+		(pin "1")
+		(instances
+			(project "Jetson-AI-Cam-CopperPilot"
+				(path "/9df9f3e2-e127-4935-b743-4d95c8ce9b2e/00000000-0000-0000-0000-0000608dc6e9"
+					(reference "#FLG_U6_VSNS")
+					(unit 1)
+				)

Commit message: fix(phase1): resolve all schematic defects across som, usb, supply, csi, id-serial with zero ERC errors
Connections:
- net 3V3_FFC1: no longer names the net of F1.2
- net 3V3_FFC2: no longer names the net of F2.2
- no-connect marks 5 -> 7
Changed lines of the file:
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@@
 		)
 	)
-	(label "PWR_EN"
+	(global_label "PWR_EN"
+		(shape input)
 		(at 393.7 67.31 180)
 		(effects
@@
 		)
 	)
-	(global_label "3V3_FFC2"
-		(shape input)
-		(at 118.745 216.535 0)
-		(fields_autoplaced yes)
-		(effects
-			(font
-				(size 1.27 1.27)
-			)
-			(justify left)
-		)
-		(property "Intersheetrefs" "${INTERSHEET_REFS}"
-			(at 130.2011 216.4556 0)
-			(hide yes)
-			(show_name no)
-			(do_not_autoplace no)
-			(effects
-				(font
-					(size 1.27 1.27)
-				)
-				(justify left)
-			)
-		)
-	)
+	(no_connect (at 118.745 216.535))
 	(global_label "VIN"
 		(shape input)
@@
 		)
 	)
-	(global_label "3V3_FFC1"
-		(shape input)
-		(at 117.475 190.5 0)
-		(fields_autoplaced yes)
-		(effects
-			(font
-				(size 1.27 1.27)
-			)
-			(justify left)
-		)
-		(property "Intersheetrefs" "${INTERSHEET_REFS}"
-			(at 128.9311 190.4206 0)
-			(hide yes)
-			(show_name no)
-			(do_not_autoplace no)
-			(effects
-				(font
-					(size 1.27 1.27)
-				)
-				(justify left)
-			)
-		)
-	)
+	(no_connect (at 117.475 190.5))
 	(global_label "VIN"
 		(shape input)

Commit message: fix(schematic): resolve electrical omissions, CSI pairs, CAN power, DNP flags, and ERC stubs
Parts:
- C23, F1, L5, U1: now not fitted; now left out of the parts list
Changed lines of the file:
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@@
 		(body_style 1)
 		(exclude_from_sim no)
-		(in_bom yes)
+		(in_bom no)
 		(on_board yes)
 		(in_pos_files yes)
-		(dnp no)
+		(dnp yes)
 		(fields_autoplaced yes)
 		(property "Reference" "U1"
@@
 		(body_style 1)
 		(exclude_from_sim no)
-		(in_bom yes)
+		(in_bom no)
 		(on_board yes)
 		(in_pos_files yes)
-		(dnp no)
+		(dnp yes)
 		(fields_autoplaced yes)
 		(property "Reference" "F1"
@@
 		(body_style 1)
 		(exclude_from_sim no)
-		(in_bom yes)
+		(in_bom no)
 		(on_board yes)
 		(in_pos_files yes)
-		(dnp no)
+		(dnp yes)
 		(fields_autoplaced yes)
 		(property "Reference" "L5"
@@
 		(body_style 1)
 		(exclude_from_sim no)
-		(in_bom yes)
+		(in_bom no)
 		(on_board yes)
 		(in_pos_files yes)
-		(dnp no)
+		(dnp yes)
 		(fields_autoplaced yes)
 		(property "Reference" "C23"
@@
 	(symbol
 		(lib_id "jetson-symbols:GND")
-		(at 351.79 102.87 0)
-		(unit 1)
-		(body_style 1)
-		(exclude_from_sim no)
-		(in_bom yes)
-		(on_board yes)
-		(in_pos_files yes)
-		(dnp no)
-		(fields_autoplaced yes)
-		(property "Reference" "#GND_080"
-			(at 351.79 102.87 0)
-			(hide yes)
-			(show_name no)
-			(do_not_autoplace no)
-			(effects
-				(font
-					(size 1.27 1.27)
-				)
-				(justify left)
-			)
-		)
-		(property "Value" "GND"
-			(at 351.79 107.315 0)
-			(show_name no)
-			(do_not_autoplace no)
-			(effects
-				(font
-					(size 1.27 1.27)
-				)
-			)
-		)
-		(property "Footprint" ""
-			(at 351.79 102.87 0)
-			(hide yes)
-			(show_name no)
-			(do_not_autoplace no)
-			(effects
-				(font
-					(size 1.27 1.27)
-				)
-				(justify left)
-			)
-		)
-		(property "Datasheet" ""
-			(at 351.79 102.87 0)
-			(hide yes)
-			(show_name no)
-			(do_not_autoplace no)
-			(effects
-				(font
-					(size 1.27 1.27)
-				)
-				(justify left)
-			)
-		)
-		(property "Description" ""
-			(at 351.79 102.87 0)
-			(show_name no)
-			(do_not_autoplace no)
-			(effects
-				(font
-					(size 1.27 1.27)
-				)
-			)
-		)
-		(property "License" "Apache-2.0"
-			(at 360.68 113.03 0)
-			(hide yes)
-			(show_name no)
-			(do_not_autoplace no)
-			(effects
-				(font
-					(size 1.27 1.27)
-					(thickness 0.15)
-				)
-				(justify left bottom)
-			)
-		)
-		(pin "1"
-		)
-		(instances
-			(project "Jetson-AI-Cam-CopperPilot"
-				(path "/9df9f3e2-e127-4935-b743-4d95c8ce9b2e/00000000-0000-0000-0000-0000608dc6e9"
-					(reference "#GND_080")
-					(unit 1)
-				)
-			)
-		)
-	)
-	(symbol
-		(lib_id "jetson-symbols:GND")
 		(at 240.03 73.66 0)
 		(unit 1)
@@
 		)
 		(stroke
-			(width 0)
-			(type default)
-		)
-	)	(wire
-		(pts
-			(xy 351.79 100.33) (xy 351.79 102.87)
-		)
-		(stroke
