File: supply.kicad_sch (KiCad schematic)
At the start: 86 parts, among them IC12 74HC00_TSSOP, IC13 SN74LVC1G126_SC-70, IC4 TPS7A0518P_SOT23-5, J12 Molex_PicoBlade_1x4_0533980471, J4 Conn_01x02, T3 BSS138PW, U1 LM3671MF-3.3_SOT, U2 LM62440-Q1, U3 SN74LXC1T45DBVR, U5 LM3671MF-3.3_SOT, U6 SIC477ED-T1-GE3

Commit message: feat(release): resolve all ERC/DRC/parity issues, complete 8-layer routing, and generate JLCPCB fab outputs
Resolve all schematic ERC violations, PCB DRC errors/warnings, schematic-to-PCB parity mismatches, and LCSC BOM/CPL fields, and package 8-layer Gerbers, drills, BOM, and CPL for JLCPCB manufacturing.

Co-Authored-By: CopperPilot <noreply@copperpilot.ai>
Parts:
- removed C16, C18, C60: C_2u2_0402, jetson-footprints:C_0402_1005Metric, symbol jetson-symbols:C_2u2_0402
- removed C17, C19, C21, C22: C_10u_1206_50V, jetson-footprints:C_1206_3216Metric, symbol jetson-symbols:C_10u_1206_50V
- removed C20, C59, C64: C_47u_0805, jetson-footprints:C_0805_2012Metric, symbol jetson-symbols:C_47u_0805
- removed C23, C55, C63, C81: C_10u_0603, jetson-footprints:C_0603_1608Metric, symbol jetson-symbols:C_10u_0603
- removed C24: C_6p_0402, jetson-footprints:C_0402_1005Metric, symbol jetson-symbols:C_6p_0402
- removed C25: C_10u_0805, jetson-footprints:C_0805_2012Metric, symbol jetson-symbols:C_10u_0805
- removed C28: C_270p_25V_0402, jetson-footprints:C_0402_1005Metric, symbol jetson-symbols:C_270p_25V_0402
- removed C41: C_47n_0402, jetson-footprints:C_0402_1005Metric, symbol jetson-symbols:C_47n_0402
- removed C56: C_100n_50V_0402, jetson-footprints:C_0402_1005Metric, symbol jetson-symbols:C_100n_50V_0402
- removed C57, C71, C83, C86, C88, C89: C_100n_0402, jetson-footprints:C_0402_1005Metric, symbol jetson-symbols:C_100n_0402
- removed C58: C_33n_0402, jetson-footprints:C_0402_1005Metric, symbol jetson-symbols:C_33n_0402
- removed C61, C82: C_1n2_50V_0402, jetson-footprints:C_0402_1005Metric, symbol jetson-symbols:C_1n2_50V_0402
- removed C65, C84, C87: C_1u_0402, jetson-footprints:C_0402_1005Metric, symbol jetson-symbols:C_1u_0402
- removed C85: C_4u7_0603, jetson-footprints:C_0603_1608Metric, symbol jetson-symbols:C_4u7_0603
- removed D1, D9: ESD5B5_0ST1G, jetson-footprints:SOD-523_NP, symbol jetson-symbols:ESD5B5_0ST1G
- removed D13: 1N4148WS, jetson-footprints:D_SOD-323F, symbol jetson-symbols:1N4148WS
- removed D14: SMBJ33A, jetson-footprints:D_SMB, symbol jetson-symbols:SMBJ33A
- removed F1, F2: F_1.25A_0603, jetson-footprints:F_0603_1608Metric, symbol jetson-symbols:F_1.25A_0603
- removed F3: F_12A_1206, jetson-footprints:F_1206_3216Metric, symbol jetson-symbols:F_12A_1206
- removed FB1: FB_10Z_10A_WE-MPSB_1206, jetson-footprints:FB_1206_3216Metric, symbol jetson-symbols:FB_10Z_10A_WE-MPSB_1206
- removed FB3: FB_180Z_3.1A_WE-MPSB_0805, jetson-footprints:FB_0805_2012Metric, symbol jetson-symbols:FB_180Z_3.1A_WE-MPSB_0805
- removed IC12: 74HC00_TSSOP, jetson-footprints:TSSOP-14_4.4x5mm_P0.65mm, symbol jetson-symbols:74HC00_TSSOP
- removed IC13: SN74LVC1G126_SC-70, jetson-footprints:SC-70-5, symbol jetson-symbols:SN74LVC1G126_SC-70
- removed IC4: TPS7A0518P_SOT23-5, jetson-footprints:SOT-23-5, symbol jetson-symbols:TPS7A0518P_SOT23-5
- removed J12: Molex_PicoBlade_1x4_0533980471, jetson-footprints:Conn_Molex_PicoBlade_1x4_0533980471, symbol jetson-symbols:Molex_PicoBlade_1x4_0533980471
- removed J4: Conn_01x02, jetson-footprints:PinHeader_1x02_P2.54mm_Vertical, symbol jetson-symbols:Conn_01x02
- removed L1: L_2u2_8A_Coilcraft-XFL4020, jetson-footprints:L_Coilcraft-XFL4020, symbol jetson-symbols:L_2u2_8A_Coilcraft-XFL4020
- removed L4: L_3u3_9.2A_Vishay-IHLP-3232DZ-01, jetson-footprints:L_Vishay-IHLP3232DZ, symbol jetson-symbols:L_3u3_9.2A_Vishay-IHLP-3232DZ-01
- removed L5, L6: L_2u2_1.6A_1210, jetson-footprints:L_1210_3225Metric, symbol jetson-symbols:L_2u2_1.6A_1210
- removed R117: R_52k3_0402, jetson-footprints:R_0402_1005Metric, symbol jetson-symbols:R_52k3_0402
- removed R118, R91, R96: R_100k_0402, jetson-footprints:R_0402_1005Metric, symbol jetson-symbols:R_100k_0402
- removed R119: R_44k2_0402, jetson-footprints:R_0402_1005Metric, symbol jetson-symbols:R_44k2_0402
- removed R120, R39, R44, R46, R52, R95: R_10k_0402, jetson-footprints:R_0402_1005Metric, symbol jetson-symbols:R_10k_0402
- removed R130, R48, R76, R92, R93: R_0R_0402, jetson-footprints:R_0402_1005Metric, symbol jetson-symbols:R_0R_0402
- removed R16, R36, R45, R87: R_1k_0402, jetson-footprints:R_0402_1005Metric, symbol jetson-symbols:R_1k_0402
- removed R70: R_100R_0402, jetson-footprints:R_0402_1005Metric, symbol jetson-symbols:R_100R_0402
- removed R74: R_2k_0402, jetson-footprints:R_0402_1005Metric, symbol jetson-symbols:R_2k_0402
- removed R75: R_316k_0402, jetson-footprints:R_0402_1005Metric, symbol jetson-symbols:R_316k_0402
- removed R77: R_60k4_0402, jetson-footprints:R_0402_1005Metric, symbol jetson-symbols:R_60k4_0402
- removed R84, R86: R_200k_0402, jetson-footprints:R_0402_1005Metric, symbol jetson-symbols:R_200k_0402
- removed R85: R_470k_0402, jetson-footprints:R_0402_1005Metric, symbol jetson-symbols:R_470k_0402
- removed R89: R_3R3_0402, jetson-footprints:R_0402_1005Metric, symbol jetson-symbols:R_3R3_0402
- removed R90: R_26k7_0402, jetson-footprints:R_0402_1005Metric, symbol jetson-symbols:R_26k7_0402
- removed R94: R_8k66_0402, jetson-footprints:R_0402_1005Metric, symbol jetson-symbols:R_8k66_0402
- removed T3: BSS138PW, jetson-footprints:SC70-3, symbol jetson-symbols:BSS138PW
- removed U1, U5: LM3671MF-3.3_SOT, jetson-footprints:SOT-23-5, symbol jetson-symbols:LM3671MF-3.3_SOT
- removed U2: LM62440-Q1, jetson-footprints:VQFN-HR-14_3.5x4mm, symbol jetson-symbols:LM62440-Q1
- removed U3: SN74LXC1T45DBVR, jetson-footprints:SOT-23-6, symbol jetson-symbols:SN74LXC1T45DBVR
- removed U6: SIC477ED-T1-GE3, jetson-footprints:SIC47XED-T1-GE3, symbol jetson-symbols:SIC477ED-T1-GE3
Connections:
- no-connect marks 7 -> 0
Other:
- note removed: "#PWR_RST"
- note removed: "0.8V typ"
- note removed: "12A"
- note removed: "1MHz"
- note removed: "3V3 DC/DC"
- note removed: "3V3 FFC 1&2"
- note removed: "3V3/3.5A"
- note removed: "52k3 -> 4.98V"
- note removed: "52k5 -> 5.0V"
- note removed: "5V DC/DC"
- note removed: "5V/8A"
- note removed: "9...36 VDC"
- note removed: "FAN 5V"
- note removed: "Note: Place close to the feedback resistors"
- note removed: "Note: SIC477 can be substituted with SIC472. If so: R75, R77, R94, C28, C61, C82 are populated, R76, R93 are DNP"
- note removed: "Power Supply"
- note removed: "Power input"
- note removed: "Power save mode enabled, VDD, VDRVPre-reg on"
- note removed: "Power sequencer"
- note removed: "R_FB_H = R_FB_L * (V_OUT - V_FB) / V_FB 10k * (5 - 0.8) / 0.8 = 52K5"
- note removed: "System 1V8"
- note removed: "Text"

Commit message: fix(sch): resolve all symbol, label, property, and syntax collisions on Supply sheet (Page 6)
Fix unquoted COMP pin name in SIC477ED-T1-GE3, relocate #FLG0313 and #FLG0312 PWR_FLAGs, move R93/C61/R96/R76/R44/R70/L1/U1/U5/IC4/U3 properties out of bodies and wires, fix R117 table box, hide J4 duplicate Description, remove duplicate PWR_EN label and J12 MP1/MP2 no_connect conflicts, and delete stray off-sheet artifacts.

Co-Authored-By: CopperPilot <noreply@copperpilot.ai>
Parts:
- added C16, C18, C60: C_2u2_0402, jetson-footprints:C_0402_1005Metric, symbol jetson-symbols:C_2u2_0402
- added C17, C19, C21, C22: C_10u_1206_50V, jetson-footprints:C_1206_3216Metric, symbol jetson-symbols:C_10u_1206_50V
- added C20, C59, C64: C_47u_0805, jetson-footprints:C_0805_2012Metric, symbol jetson-symbols:C_47u_0805
- added C23, C55, C63, C81: C_10u_0603, jetson-footprints:C_0603_1608Metric, symbol jetson-symbols:C_10u_0603
- added C24: C_6p_0402, jetson-footprints:C_0402_1005Metric, symbol jetson-symbols:C_6p_0402
- added C25: C_10u_0805, jetson-footprints:C_0805_2012Metric, symbol jetson-symbols:C_10u_0805
- added C28: C_270p_25V_0402, jetson-footprints:C_0402_1005Metric, symbol jetson-symbols:C_270p_25V_0402
- added C41: C_47n_0402, jetson-footprints:C_0402_1005Metric, symbol jetson-symbols:C_47n_0402
- added C56: C_100n_50V_0402, jetson-footprints:C_0402_1005Metric, symbol jetson-symbols:C_100n_50V_0402
- added C57, C71, C83, C86, C88, C89: C_100n_0402, jetson-footprints:C_0402_1005Metric, symbol jetson-symbols:C_100n_0402
- added C58: C_33n_0402, jetson-footprints:C_0402_1005Metric, symbol jetson-symbols:C_33n_0402
- added C61, C82: C_1n2_50V_0402, jetson-footprints:C_0402_1005Metric, symbol jetson-symbols:C_1n2_50V_0402
- added C65, C84, C87: C_1u_0402, jetson-footprints:C_0402_1005Metric, symbol jetson-symbols:C_1u_0402
- added C85: C_4u7_0603, jetson-footprints:C_0603_1608Metric, symbol jetson-symbols:C_4u7_0603
- added D1, D9: ESD5B5_0ST1G, jetson-footprints:SOD-523_NP, symbol jetson-symbols:ESD5B5_0ST1G
- added D13: 1N4148WS, jetson-footprints:D_SOD-323F, symbol jetson-symbols:1N4148WS
- added D14: SMBJ33A, jetson-footprints:D_SMB, symbol jetson-symbols:SMBJ33A
- added F1, F2: F_1.25A_0603, jetson-footprints:F_0603_1608Metric, symbol jetson-symbols:F_1.25A_0603
- added F3: F_12A_1206, jetson-footprints:F_1206_3216Metric, symbol jetson-symbols:F_12A_1206
- added FB1: FB_10Z_10A_WE-MPSB_1206, jetson-footprints:FB_1206_3216Metric, symbol jetson-symbols:FB_10Z_10A_WE-MPSB_1206
- added FB3: FB_180Z_3.1A_WE-MPSB_0805, jetson-footprints:FB_0805_2012Metric, symbol jetson-symbols:FB_180Z_3.1A_WE-MPSB_0805
- added IC12: 74HC00_TSSOP, jetson-footprints:TSSOP-14_4.4x5mm_P0.65mm, symbol jetson-symbols:74HC00_TSSOP
- added IC13: SN74LVC1G126_SC-70, jetson-footprints:SC-70-5, symbol jetson-symbols:SN74LVC1G126_SC-70
- added IC4: TPS7A0518P_SOT23-5, jetson-footprints:SOT-23-5, symbol jetson-symbols:TPS7A0518P_SOT23-5
- added J12: Molex_PicoBlade_1x4_0533980471, jetson-footprints:Conn_Molex_PicoBlade_1x4_0533980471, symbol jetson-symbols:Molex_PicoBlade_1x4_0533980471
- added J4: Conn_01x02, jetson-footprints:PinHeader_1x02_P2.54mm_Vertical, symbol jetson-symbols:Conn_01x02
- added L1: L_2u2_8A_Coilcraft-XFL4020, jetson-footprints:L_Coilcraft-XFL4020, symbol jetson-symbols:L_2u2_8A_Coilcraft-XFL4020
- added L4: L_3u3_9.2A_Vishay-IHLP-3232DZ-01, jetson-footprints:L_Vishay-IHLP3232DZ, symbol jetson-symbols:L_3u3_9.2A_Vishay-IHLP-3232DZ-01
- added L5, L6: L_2u2_1.6A_1210, jetson-footprints:L_1210_3225Metric, symbol jetson-symbols:L_2u2_1.6A_1210
- added R117: R_52k3_0402, jetson-footprints:R_0402_1005Metric, symbol jetson-symbols:R_52k3_0402
- added R118, R91, R96: R_100k_0402, jetson-footprints:R_0402_1005Metric, symbol jetson-symbols:R_100k_0402
- added R119: R_44k2_0402, jetson-footprints:R_0402_1005Metric, symbol jetson-symbols:R_44k2_0402
- added R120, R39, R44, R46, R52, R95: R_10k_0402, jetson-footprints:R_0402_1005Metric, symbol jetson-symbols:R_10k_0402
- added R130, R48, R76, R92, R93: R_0R_0402, jetson-footprints:R_0402_1005Metric, symbol jetson-symbols:R_0R_0402
- added R16, R36, R45, R87: R_1k_0402, jetson-footprints:R_0402_1005Metric, symbol jetson-symbols:R_1k_0402
- added R70: R_100R_0402, jetson-footprints:R_0402_1005Metric, symbol jetson-symbols:R_100R_0402
- added R74: R_2k_0402, jetson-footprints:R_0402_1005Metric, symbol jetson-symbols:R_2k_0402
- added R75: R_316k_0402, jetson-footprints:R_0402_1005Metric, symbol jetson-symbols:R_316k_0402
- added R77: R_60k4_0402, jetson-footprints:R_0402_1005Metric, symbol jetson-symbols:R_60k4_0402
- added R84, R86: R_200k_0402, jetson-footprints:R_0402_1005Metric, symbol jetson-symbols:R_200k_0402
- added R85: R_470k_0402, jetson-footprints:R_0402_1005Metric, symbol jetson-symbols:R_470k_0402
- added R89: R_3R3_0402, jetson-footprints:R_0402_1005Metric, symbol jetson-symbols:R_3R3_0402
- added R90: R_26k7_0402, jetson-footprints:R_0402_1005Metric, symbol jetson-symbols:R_26k7_0402
- added R94: R_8k66_0402, jetson-footprints:R_0402_1005Metric, symbol jetson-symbols:R_8k66_0402
- added T3: BSS138PW, jetson-footprints:SC70-3, symbol jetson-symbols:BSS138PW
- added U1, U5: LM3671MF-3.3_SOT, jetson-footprints:SOT-23-5, symbol jetson-symbols:LM3671MF-3.3_SOT
- added U2: LM62440-Q1, jetson-footprints:VQFN-HR-14_3.5x4mm, symbol jetson-symbols:LM62440-Q1
- added U3: SN74LXC1T45DBVR, jetson-footprints:SOT-23-6, symbol jetson-symbols:SN74LXC1T45DBVR
- added U6: SIC477ED-T1-GE3, jetson-footprints:SIC47XED-T1-GE3, symbol jetson-symbols:SIC477ED-T1-GE3
Connections:
- new net: IC12.10 (3B), IC12.11 (~{4Y}), IC12.9 (3A)
- new net: IC12.2 (1B), IC12.6 (~{2Y}), R16.2
- new net: IC12.8 (~{3Y}), R130.2
- new net: F3.1, J4.1 (Pin_1)
- new net: IC4.3 (EN), R92.2
- new net: C23.1, F1.1, L5.2, U1.4 (FB)
- new net: C55.1, F2.1, L6.2, U5.4 (FB)
- new net: C57.1, R89.1
- new net: R39.2, U1.3 (EN)
- new net: L5.1, U1.5 (SW)
- new net: R52.2, U5.3 (EN)
- new net: L6.1, U5.5 (SW)
- new net: C61.1, R93.1, U6.20 (VOUT)
- new net: R70.1, U2.13 (RBOOT)
- new net: C24.2, R45.1
- new net: C28.1, R75.2
- new net #RESET: R39.1, R44.1, R52.1, R92.1
- new net #SHUTDOWN_REQ: IC12.4 (2A), R86.2
- new net 1V8_SYS: C65.1, C86.1, IC4.5 (VOUT), R95.1, T3.1 (G), U3.1 (VCCA), U3.5 (DIR)
- new net 3V3_EN: R44.2, U2.7 (EN)
- new net 3V3_FB: R118.2, R119.1, R45.2, R48.2, U2.4 (FB)
- new net 3V3_R_C_BOOT: C89.2, R70.2, U2.14 (CBOOT)
- new net 3V3_SW: C89.1, L1.1, U2.10 (SW)
- new net 3V3_SYS: C20.1, C24.1, C25.1, D1.2 (A), L1.2, R118.1, R48.1, U2.1 (BIAS)
- new net 3V3_VCC: C87.1, U2.2 (VCC)
- new net 3V3_VIN: C19.1, C21.1, FB3.2, U2.12 (VIN), U2.8 (VIN)
- new net 5V0_SYS: C16.1, C18.1, C59.1, C60.1, C64.1, C71.1, C81.1, C82.2, C83.1, C88.1, D9.2 (A), IC12.14 (VCC), IC13.1 (OE), IC13.5 (VCC), IC4.1 (VIN), J12.2, L4.2, R117.1, R16.1, R36.1, R46.1, R84.1, R86.1, R93.2, U1.1 (V_{IN}), U3.6 (VCCB), U5.1 (V_{IN})
- new net 5V_BOOT: C57.2, U6.4 (BOOT)
- new net 5V_COMP: R75.1, U6.21 (~{COMP})
- new net 5V_EN: R91.1, U6.3 (EN)
- new net 5V_FB: R117.2, R120.1, U6.22 (V_{FB})
- new net 5V_FSW: R90.1, U6.24 (f_{SW})
- new net 5V_ILIM: R76.2, R77.1, U6.25 (I_{LIMIT})
- new net 5V_MODE: R74.1, U6.27 (MODE)
- new net 5V_PHASE: R89.2, U6.5 (PHASE), U6.6 (PHASE)
- new net 5V_SNS: C61.2, C82.1, R94.2
- new net 5V_SS: C58.1, U6.19 (SS)
- new net 5V_SW: L4.1, R94.1, U6.12 (SW), U6.13 (SW), U6.14 (SW)
- new net 5V_VIN: C17.1, C22.1, C56.1, FB1.2, R91.2, U6.1 (V_{CIN}), U6.7 (V_{IN}), U6.8 (V_{IN})
- new net FAN_PMW_5V: J12.4, U3.4 (B)
- new net FAN_PWM: U3.3 (A)
- new net FAN_TACH: R95.2, T3.2 (S)
- new net FAN_TACH_5V: J12.3, R46.2, T3.3 (D)
- new net GND: C16.2, C17.2, C18.2, C19.2, C20.2, C21.2, C22.2, C23.2, C25.2, C28.2, C41.2, C55.2, C56.2, C58.2, C59.2, C60.2, C63.2, C64.2, C65.2, C71.2, C81.2, C83.2, C84.2, C85.2, C86.2, C87.2, C88.2, D1.1 (C), D14.2 (A), D9.1 (C), IC12.7 (GND), IC13.3 (GND), IC4.2 (GND), J12.1, J12.MP1, J12.MP2, J4.2 (Pin_2), R119.2, R120.2, R74.2, R77.2, R90.2, U1.2 (GND), U2.11 (PGND), U2.3 (AGND), U2.6 (MODE), U2.9 (PGND), U3.2 (GND), U5.2 (GND), U6.10 (PGND), U6.11 (PGND), U6.17 (PGND), U6.23 (AGND), U6.28 (AGND), U6.9 (PGND)
- new net PWR_EN: IC13.4 (Y), R130.1
- new net PWR_GOOD: R87.1, R96.1, U6.2 (P_{GOOD})
- new net Q: D13.1 (C), IC12.3 (~{1Y}), IC12.5 (2B), R36.2, R85.1
- new net QDEL: C63.1, D13.2 (A), IC12.12 (4A), IC12.13 (4B), IC13.2 (A), R85.2, R87.2
- new net VDD_5V_DCDC: C84.1, R76.1, R96.2, U6.26 (V_{DD})
- new net VDRV_5V_DCDC: C85.1, U6.16 (V_{DRV})
- new net VIN: D14.1 (C), F3.2, FB1.1, FB3.1
- new net \~{PWR_SET}: C41.1, IC12.1 (1A), R84.2
- no-connect marks 0 -> 5
Other:
- note added: "#PWR_RST"
- note added: "0.8V typ"
- note added: "12A"
- note added: "1MHz"
- note added: "3V3 DC/DC"
- note added: "3V3 FFC 1&2"
- note added: "3V3/3.5A"
- note added: "52k3 -> 4.98V"
- note added: "52k5 -> 5.0V"
- note added: "5V DC/DC"
- note added: "5V/8A"
- note added: "9...36 VDC"
- note added: "FAN 5V"
- note added: "Note: Place close to the feedback resistors"
- note added: "Note: SIC477 can be substituted with SIC472. If so: R75, R77, R94, C28, C61, C82 are populated, R76, R93 are DNP"
- note added: "Power Supply"
- note added: "Power input"
- note added: "Power save mode enabled, VDD, VDRV Pre-reg on"
- note added: "Power sequencer"
- note added: "R_FB_H = R_FB_L * (V_OUT - V_FB) / V_FB 10k * (5 - 0.8) / 0.8 = 52K5"
- note added: "System 1V8"
