File: supply.kicad_sch (KiCad schematic)
At the start: 86 parts, among them IC12 74HC00_TSSOP, IC13 SN74LVC1G126_SC-70, IC4 TPS7A0518P_SOT23-5, J12 Molex_PicoBlade_1x4_0533980471, J4 Conn_01x02, T3 BSS138PW, U1 LM3671MF-3.3_SOT, U2 LM62440-Q1, U3 SN74LXC1T45DBVR, U5 LM3671MF-3.3_SOT, U6 SIC477ED-T1-GE3

Commit message: fix(sch): configure U2 3.3V buck feedback divider and tune POWER_EN boot delay
Set R48 to DNP and populate R118/R119/R45/C24 divider network to ensure 3.3V regulation from LMQ62440 1.0V internal reference. Retune R85 to 10k for 100ms POWER_EN boot delay.

Co-Authored-By: CopperPilot <noreply@copperpilot.ai>
Parts:
- C24, R118, R45: now fitted; now in the parts list
- R119: LCSC (none) -> C137980; now fitted; now in the parts list
- R48: now not fitted; now left out of the parts list
- R85: value R_470k_0402 -> R_10k_0402; symbol jetson-symbols:R_470k_0402 -> jetson-symbols:R_10k_0402; LCSC C25790 -> C25744; MPN CR0402-FX-4703GLF -> CR0402-FX-1002GLF; Val 470k -> 10k
Changed lines of the file:
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@@
 		(body_style 1)
 		(exclude_from_sim no)
-		(in_bom yes)
+		(in_bom no)
 		(on_board yes)
 		(in_pos_files yes)
-		(dnp no)
+		(dnp yes)
 		(property "Reference" "R48"
 			(at 150.495 140.335 90)
@@
 		(body_style 1)
 		(exclude_from_sim no)
-		(in_bom no)
+		(in_bom yes)
 		(on_board yes)
 		(in_pos_files yes)
-		(dnp yes)
+		(dnp no)
 		(property "Reference" "R118"
 			(at 140.97 140.335 90)
@@
 		(body_style 1)
 		(exclude_from_sim no)
-		(in_bom no)
+		(in_bom yes)
 		(on_board yes)
 		(in_pos_files yes)
-		(dnp yes)
+		(dnp no)
 		(property "Reference" "R119"
 			(at 140.97 153.035 90)
@@
 			)
 		)
+		(property "LCSC" "C137980"
+			(at 0 0 0)
+			(effects
+				(font
+					(size 1.27 1.27)
+				)
+				(hide yes)
+			)
+		)
 		(pin "1"
 		)
@@
 	)
 	(symbol
-		(lib_id "jetson-symbols:R_470k_0402")
+		(lib_id "jetson-symbols:R_10k_0402")
 		(at 330.2 67.31 0)
 		(unit 1)
@@
 			)
 		)
-		(property "Value" "R_470k_0402"
+		(property "Value" "R_10k_0402"
 			(at 330.2 71.12 0)
 			(hide yes)
@@
 			)
 		)
-		(property "MPN" "CR0402-FX-4703GLF"
+		(property "MPN" "CR0402-FX-1002GLF"
 			(at 335.28 59.69 0)
 			(hide yes)
@@
 			)
 		)
-		(property "Val" "470k"
+		(property "Val" "10k"
 			(at 332.74 69.85 0)
 			(show_name no)
@@
 		)
 		(property "License" "Apache-2.0"
-			(at 350.52 92.71 0)
+			(at 304.8 87.63 0)
 			(hide yes)
 			(show_name no)
@@
 			)
 		)
-		(property "LCSC" "C25790"
+		(property "LCSC" "C25744"
 			(at 0 0 0)
 			(effects
@@
 		(body_style 1)
 		(exclude_from_sim no)
-		(in_bom no)
+		(in_bom yes)
 		(on_board yes)
 		(in_pos_files yes)
-		(dnp yes)
+		(dnp no)
 		(property "Reference" "R45"
 			(at 131.445 144.145 90)
@@
 		(body_style 1)
 		(exclude_from_sim no)
-		(in_bom no)
+		(in_bom yes)
 		(on_board yes)
 		(in_pos_files yes)
-		(dnp yes)
+		(dnp no)
 		(property "Reference" "C24"
 			(at 132.715 137.795 90)
