File: som.kicad_sch (KiCad schematic)
At the start: 30 parts, among them J10 Conn_FFC_Molex_5051101097, J15 Bus_DDR4_SODIMM_CUSTOM_Jetson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, M2 Jetson-Nano, T2 BSS138PW, T4 BSS138PW, T5 BSS138PW

Commit message: fix(sch): resolve all PWR_FLAG, label, and differential-corridor collisions on Display sheet (Page 5)
Remove duplicate TMDS_HPD label on J15E, relocate colliding PWR_FLAG symbols on J1/J2/IC2/top-left and hide flag text, move C73-C80/R1-R10/C39-C45/R98-R99 properties out of differential wire corridors, clean up R31/R32/T1, and delete stray off-sheet artifacts.

Co-Authored-By: CopperPilot <noreply@copperpilot.ai>
Changed lines of the file:
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@@
 		)
 		(property "Value" "Spacer_Drill3.7mm_H6mm_9774060151R"
-			(at 355.6 252.73 0)
+			(at 355.6 248.92 0)
+			(hide yes)
 			(show_name no)
 			(do_not_autoplace no)
@@
 		(dnp yes)
 		(property "Reference" "SP2"
-			(at 355.6 213.36 0)
+			(at 355.6 218.44 0)
 			(show_name no)
 			(do_not_autoplace no)
@@
 		)
 		(property "Value" "Spacer_Drill3.7mm_H6mm_9774060151R"
-			(at 355.6 215.9 0)
+			(at 355.6 220.98 0)
+			(hide yes)
 			(show_name no)
 			(do_not_autoplace no)
@@
 		(fields_autoplaced yes)
 		(property "Reference" "C103"
-			(at 273.05 55.88 0)
+			(at 271.78 56.515 0)
 			(effects (font (size 1.27 1.27)) (justify left))
 		)
@@
 		(fields_autoplaced yes)
 		(property "Reference" "C104"
-			(at 280.67 55.88 0)
+			(at 278.13 56.515 0)
 			(effects (font (size 1.27 1.27)) (justify left))
 		)
@@
 	)
 	(label "PMIC_BBAT"
-		(at 100.33 50.8 0)
+		(at 80.01 50.8 0)
 		(effects
 			(font
@@
 	)
 	(wire
-		(pts (xy 74.93 50.8) (xy 100.33 50.8))
+		(pts (xy 74.93 50.8) (xy 80.01 50.8))
 		(stroke
 			(width 0)

Commit message: fix(bom): update LCSC procurement part numbers and SMT assembly flags
Reconcile LCSC part numbers with physical land patterns and active stock:
- J11 USB-C: C456013 (24-pin SuperSpeed receptacle matching Wurth 632723300011)
- J15 SODIMM: C2766246 (TE 2309413-1 260-pin socket)
- J2 Mini-DP: C574827 (TE 2129320-3)
- J1 Micro-HDMI: C563878 (Molex 467651001)
- J5, J9 Micro-USB: C132560 (Molex 473460001)
- REC1, RST1, USR1: C2886925 (E-Switch TL3340AF160QG)
- BAT1: set DNP for SMT reflow to prevent thermal rupture in 260C oven

Co-Authored-By: CopperPilot <noreply@copperpilot.ai>
Parts:
- BAT1: now not fitted; now left out of the parts list
- J15: LCSC C429199 -> C2766246
- REC1, RST1, USR1: LCSC C140844 -> C2886925
Changed lines of the file:
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@@
 			)
 		)
-		(property "LCSC" "C429199"
+		(property "LCSC" "C2766246"
 			(at 0 0 0)
 			(effects
@@
 			)
 		)
-		(property "LCSC" "C429199"
+		(property "LCSC" "C2766246"
 			(at 0 0 0)
 			(effects
@@
 			)
 		)
-		(property "LCSC" "C429199"
+		(property "LCSC" "C2766246"
 			(at 0 0 0)
 			(effects
@@
 			)
 		)
-		(property "LCSC" "C429199"
+		(property "LCSC" "C2766246"
 			(at 0 0 0)
 			(effects
@@
 			)
 		)
-		(property "LCSC" "C429199"
+		(property "LCSC" "C2766246"
 			(at 0 0 0)
 			(effects
@@
 			)
 		)
-		(property "LCSC" "C140844"
+		(property "LCSC" "C2886925"
 			(at 0 0 0)
 			(effects
@@
 		(body_style 1)
 		(exclude_from_sim no)
-		(in_bom yes)
+		(in_bom no)
 		(on_board yes)
 		(in_pos_files yes)
-		(dnp no)
+		(dnp yes)
 		(fields_autoplaced yes)
 		(property "Reference" "BAT1"
@@
 			)
 		)
-		(property "LCSC" "C140844"
+		(property "LCSC" "C2886925"
 			(at 0 0 0)
 			(effects
@@
 			)
 		)
-		(property "LCSC" "C140844"
+		(property "LCSC" "C2886925"
 			(at 0 0 0)
 			(effects
