File: usb-debug.kicad_sch (KiCad schematic)
At the start: 83 parts, among them IC1 NCP380LSNAJAAT1G, IC15 TPS7A0518P_SOT23-5, IC3 NCP380LSNAJAAT1G, IC5 FT232R_QFN, IC7 HD3SS3220RNH, J11 USB-C_WE_632723300011, J5 USB-Micro-B_Molex_473460001, J9 USB-Micro-B_Molex_473460001, T6 BSS138PW, T7 BSS138PW, T9 BSS138PW, U8 74LVC1G07_SOT-753

Commit message: fix(bom): update LCSC procurement part numbers and SMT assembly flags
Reconcile LCSC part numbers with physical land patterns and active stock:
- J11 USB-C: C456013 (24-pin SuperSpeed receptacle matching Wurth 632723300011)
- J15 SODIMM: C2766246 (TE 2309413-1 260-pin socket)
- J2 Mini-DP: C574827 (TE 2129320-3)
- J1 Micro-HDMI: C563878 (Molex 467651001)
- J5, J9 Micro-USB: C132560 (Molex 473460001)
- REC1, RST1, USR1: C2886925 (E-Switch TL3340AF160QG)
- BAT1: set DNP for SMT reflow to prevent thermal rupture in 260C oven

Co-Authored-By: CopperPilot <noreply@copperpilot.ai>
Parts:
- J11: LCSC C393939 -> C456013
- J5, J9: LCSC C132563 -> C132560
Changed lines of the file:
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@@
 			)
 		)
-		(property "LCSC" "C132563"
+		(property "LCSC" "C132560"
 			(at 0 0 0)
 			(effects
@@
 			)
 		)
-		(property "LCSC" "C393939"
+		(property "LCSC" "C456013"
 			(at 0 0 0)
 			(effects
@@
 			)
 		)
-		(property "LCSC" "C132563"
+		(property "LCSC" "C132560"
 			(at 0 0 0)
 			(effects
